File: High speed isolator.kicad_sch (KiCad schematic)
At the start: 6 parts, among them IC5 CA-IS3731LN

Commit message: adding high speed isolator
Parts:
- IC5: footprint SOIC127P600X175-16N -> SamacSys_Parts:SOIC127P600X175-16N
Changed lines of the file:
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@@
       (effects (font (size 1.27 1.27)))
     )
-    (property "Footprint" "SOIC127P600X175-16N" (at 156.845 206.045 0)
+    (property "Footprint" "SamacSys_Parts:SOIC127P600X175-16N" (at 156.845 206.045 0)
       (effects (font (size 1.27 1.27)) (justify left top) hide)
     )
@@
       (effects (font (size 1.27 1.27)))
     )
-    (property "Footprint" "SOIC127P600X175-16N" (at 157.48 145.085 0)
-      (effects (font (size 1.27 1.27)) (justify left top) hide)
-    )
+    (property "Footprint" "SamacSys_Parts:SOIC127P600X175-16N" (at 157.48 145.085 0)
+      (effects (font (size 1.27 1.27)) (justify left top) hide)
+    )
