File: MCU.kicad_sch (KiCad schematic)
At the start: 1 part, among them J4 STM32F407G-DISC1-SHIELD

Commit message: updating component & board
Connections:
- removed net VDD: J4.2 (VDD), J4.27 (VDD), J4.36 (VDD)
- no-connect marks 72 -> 75
Changed lines of the file:
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@@
   (no_connect (at 180.34 104.775))
   (no_connect (at 158.75 94.615))
+  (no_connect (at 130.81 64.135))
   (no_connect (at 129.54 114.935))
   (no_connect (at 129.54 104.775))
@@
   (no_connect (at 158.75 79.375))
   (no_connect (at 180.34 81.915))
+  (no_connect (at 106.68 64.135))
   (no_connect (at 129.54 89.535))
   (no_connect (at 158.75 114.935))
@@
   (no_connect (at 158.75 109.855))
   (no_connect (at 180.34 99.695))
+  (no_connect (at 181.61 86.995))
   (no_connect (at 158.75 92.075))
   (no_connect (at 158.75 86.995))
@@
     )
   )
-  (symbol (lib_id "power:VDD") (at 106.68 64.135 90) (unit 1)
-    (in_bom yes) (on_board yes) (dnp no) (fields_autoplaced)
-    (property "Reference" "#PWR010" (at 110.49 64.135 0)
-      (effects (font (size 1.27 1.27)) hide)
-    )
-    (property "Value" "VDD" (at 103.505 64.135 90)
-      (effects (font (size 1.27 1.27)) (justify left))
-    )
-    (property "Footprint" "" (at 106.68 64.135 0)
-      (effects (font (size 1.27 1.27)) hide)
-    )
-    (property "Datasheet" "" (at 106.68 64.135 0)
-      (effects (font (size 1.27 1.27)) hide)
-    )
-    (pin "1")
-    (instances
-      (project "Main"
-        (path "/c97a22ab-71f8-4b91-b313-15b8a3e640d7"
-          (reference "#PWR010") (unit 1)
-        )
-        (path "/c97a22ab-71f8-4b91-b313-15b8a3e640d7/9673f451-06b8-4c7c-85a7-44eae9f9c3b1"
-          (reference "#PWR02") (unit 1)
-        )
-      )
-    )
-  )
   (symbol (lib_id "power:GND") (at 106.68 89.535 270) (unit 1)
     (in_bom yes) (on_board yes) (dnp no) (fields_autoplaced)
@@
     )
   )
-  (symbol (lib_id "power:VDD") (at 130.81 64.135 270) (unit 1)
-    (in_bom yes) (on_board yes) (dnp no) (fields_autoplaced)
-    (property "Reference" "#PWR011" (at 127 64.135 0)
-      (effects (font (size 1.27 1.27)) hide)
-    )
-    (property "Value" "VDD" (at 133.985 64.135 90)
-      (effects (font (size 1.27 1.27)) (justify left))
-    )
-    (property "Footprint" "" (at 130.81 64.135 0)
-      (effects (font (size 1.27 1.27)) hide)
-    )
-    (property "Datasheet" "" (at 130.81 64.135 0)
-      (effects (font (size 1.27 1.27)) hide)
-    )
-    (pin "1")
-    (instances
-      (project "Main"
-        (path "/c97a22ab-71f8-4b91-b313-15b8a3e640d7"
-          (reference "#PWR011") (unit 1)
-        )
-        (path "/c97a22ab-71f8-4b91-b313-15b8a3e640d7/9673f451-06b8-4c7c-85a7-44eae9f9c3b1"
-          (reference "#PWR07") (unit 1)
-        )
-      )
-    )
-  )
   (symbol (lib_id "power:GND") (at 130.81 122.555 90) (unit 1)
     (in_bom yes) (on_board yes) (dnp no) (fields_autoplaced)
@@
         )
       )
-    )
-  )
-  (symbol (lib_id "power:VDD") (at 181.61 86.995 270) (unit 1)
-    (in_bom yes) (on_board yes) (dnp no) (fields_autoplaced)
-    (property "Reference" "#PWR013" (at 177.8 86.995 0)
-      (effects (font (size 1.27 1.27)) hide)
-    )
-    (property "Value" "VDD" (at 184.785 86.995 90)
-      (effects (font (size 1.27 1.27)) (justify left))
-    )
-    (property "Footprint" "" (at 181.61 86.995 0)
-      (effects (font (size 1.27 1.27)) hide)
-    )
-    (property "Datasheet" "" (at 181.61 86.995 0)
-      (effects (font (size 1.27 1.27)) hide)
-    )
-    (pin "1")
-    (instances
-      (project "Main"
-        (path "/c97a22ab-71f8-4b91-b313-15b8a3e640d7"
-          (reference "#PWR013") (unit 1)
-        )
-        (path "/c97a22ab-71f8-4b91-b313-15b8a3e640d7/9673f451-06b8-4c7c-85a7-44eae9f9c3b1"
-          (reference "#PWR016") (unit 1)
-        )
-      )

Commit message: update footprint
Parts:
- J4: footprint (none) -> Custom:STM32F407G-DISC1-SHIELD
Connections:
- net HIN_U: now also J4.17 (PE15); no longer J4.19 (PC10)
- net HIN_V: now also J4.13 (PE7); no longer J4.44 (PC11)
- net HIN_W: now also J4.18 (PC12); no longer J4.20 (PB15)
- net LIN_U: now also J4.15 (PE11); no longer J4.16 (PE13)
- net LIN_V: now also J4.14 (PE9); no longer J4.41 (PE14)
- net LIN_W: now also J4.16 (PE13); no longer J4.17 (PE15)
- removed net +3V0: J4.28 (NRST), J4.3 (GND)
- no-connect marks 75 -> 77
Changed lines of the file:
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@@
   (paper "A4")
   (no_connect (at 180.34 104.775))
+  (no_connect (at 129.54 107.315))
   (no_connect (at 158.75 94.615))
   (no_connect (at 130.81 64.135))
@@
   (no_connect (at 129.54 86.995))
   (no_connect (at 180.34 74.295))
+  (no_connect (at 107.95 107.315))
   (no_connect (at 158.75 81.915))
   (no_connect (at 129.54 109.855))
@@
   (no_connect (at 158.75 69.215))
   (no_connect (at 107.95 76.835))
-  (no_connect (at 107.95 97.155))
   (no_connect (at 129.54 69.215))
   (no_connect (at 158.75 79.375))
@@
   (no_connect (at 107.95 117.475))
   (no_connect (at 180.34 79.375))
-  (no_connect (at 107.95 94.615))
   (no_connect (at 180.34 76.835))
   (no_connect (at 129.54 97.155))
@@
   (no_connect (at 180.34 94.615))
   (no_connect (at 129.54 117.475))
+  (no_connect (at 180.34 66.675))
   (no_connect (at 180.34 92.075))
   (no_connect (at 180.34 112.395))
+  (no_connect (at 129.54 99.695))
   (no_connect (at 107.95 81.915))
   (no_connect (at 129.54 74.295))
   (no_connect (at 180.34 117.475))
   (no_connect (at 158.75 76.835))
-  (no_connect (at 107.95 104.775))
   (no_connect (at 180.34 120.015))
   (no_connect (at 129.54 112.395))
@@
   (no_connect (at 180.34 69.215))
   (no_connect (at 158.75 107.315))
+  (no_connect (at 158.75 66.675))
   (no_connect (at 107.95 112.395))
   (no_connect (at 129.54 94.615))
   (no_connect (at 180.34 102.235))
-  (no_connect (at 107.95 92.075))
   (no_connect (at 158.75 84.455))
+  (no_connect (at 107.95 109.855))
   (no_connect (at 158.75 89.535))
   (no_connect (at 107.95 71.755))
@@
     (stroke (width 0) (type default))
   )
-  (wire (pts (xy 105.41 109.855) (xy 107.95 109.855))
-    (stroke (width 0) (type default))
-  )
   (wire (pts (xy 180.34 64.135) (xy 181.61 64.135))
     (stroke (width 0) (type default))
   )
-  (wire (pts (xy 105.41 107.315) (xy 107.95 107.315))
+  (wire (pts (xy 81.915 102.235) (xy 107.95 102.235))
     (stroke (width 0) (type default))
   )
@@
     (stroke (width 0) (type default))
   )
-  (wire (pts (xy 180.34 66.675) (xy 181.61 66.675))
-    (stroke (width 0) (type default))
-  )
-  (wire (pts (xy 157.48 66.675) (xy 158.75 66.675))
-    (stroke (width 0) (type default))
-  )
-  (wire (pts (xy 105.41 99.695) (xy 107.95 99.695))
-    (stroke (width 0) (type default))
-  )
   (wire (pts (xy 157.48 61.595) (xy 158.75 61.595))
     (stroke (width 0) (type default))
@@
     (stroke (width 0) (type default))
   )
-  (wire (pts (xy 129.54 99.695) (xy 132.715 99.695))
-    (stroke (width 0) (type default))
-  )
   (wire (pts (xy 129.54 84.455) (xy 132.08 84.455))
     (stroke (width 0) (type default))
   )
+  (wire (pts (xy 81.915 97.155) (xy 107.95 97.155))
+    (stroke (width 0) (type default))
+  )
   (wire (pts (xy 180.34 86.995) (xy 181.61 86.995))
     (stroke (width 0) (type default))
@@
     (stroke (width 0) (type default))
   )
+  (wire (pts (xy 81.915 94.615) (xy 107.95 94.615))
+    (stroke (width 0) (type default))
+  )
   (wire (pts (xy 129.54 71.755) (xy 132.715 71.755))
     (stroke (width 0) (type default))
@@
     (stroke (width 0) (type default))
   )
-  (wire (pts (xy 129.54 107.315) (xy 132.08 107.315))
-    (stroke (width 0) (type default))
-  )
   (wire (pts (xy 106.68 89.535) (xy 107.95 89.535))
     (stroke (width 0) (type default))
   )
-  (wire (pts (xy 105.41 102.235) (xy 107.95 102.235))
-    (stroke (width 0) (type default))
-  )
   (wire (pts (xy 106.68 66.675) (xy 107.95 66.675))
     (stroke (width 0) (type default))
   )
+  (wire (pts (xy 81.915 99.695) (xy 107.95 99.695))
+    (stroke (width 0) (type default))
+  )
+  (wire (pts (xy 81.915 92.075) (xy 107.95 92.075))
+    (stroke (width 0) (type default))
+  )
+  (wire (pts (xy 81.915 104.775) (xy 107.95 104.775))
+    (stroke (width 0) (type default))
+  )
   (wire (pts (xy 106.68 122.555) (xy 107.95 122.555))
     (stroke (width 0) (type default))
@@
     (stroke (width 0) (type default))
   )
-  (hierarchical_label "HIN_W" (shape output) (at 105.41 109.855 180) (fields_autoplaced)
+  (hierarchical_label "HIN_W" (shape output) (at 81.915 104.775 180) (fields_autoplaced)
     (effects (font (size 1.27 1.27)) (justify right))
   )
@@
     (effects (font (size 1.27 1.27)) (justify left))
   )
-  (hierarchical_label "LIN_U" (shape output) (at 105.41 99.695 180) (fields_autoplaced)
-    (effects (font (size 1.27 1.27)) (justify right))
-  )
-  (hierarchical_label "HIN_V" (shape output) (at 132.08 107.315 0) (fields_autoplaced)
-    (effects (font (size 1.27 1.27)) (justify left))
+  (hierarchical_label "LIN_U" (shape output) (at 81.915 97.155 180) (fields_autoplaced)
+    (effects (font (size 1.27 1.27)) (justify right))
+  )
+  (hierarchical_label "HIN_V" (shape output) (at 81.915 92.075 180) (fields_autoplaced)
+    (effects (font (size 1.27 1.27)) (justify right))
   )
   (hierarchical_label "CURR_W" (shape input) (at 132.08 84.455 0) (fields_autoplaced)
     (effects (font (size 1.27 1.27)) (justify left))
   )
-  (hierarchical_label "LIN_W" (shape output) (at 105.41 102.235 180) (fields_autoplaced)
+  (hierarchical_label "LIN_W" (shape output) (at 81.915 99.695 180) (fields_autoplaced)
     (effects (font (size 1.27 1.27)) (justify right))
   )
@@
     (effects (font (size 1.27 1.27)) (justify left))
   )
-  (hierarchical_label "HIN_U" (shape output) (at 105.41 107.315 180) (fields_autoplaced)
-    (effects (font (size 1.27 1.27)) (justify right))
-  )
-  (hierarchical_label "LIN_V" (shape output) (at 132.715 99.695 0) (fields_autoplaced)
-    (effects (font (size 1.27 1.27)) (justify left))
+  (hierarchical_label "HIN_U" (shape output) (at 81.915 102.235 180) (fields_autoplaced)
+    (effects (font (size 1.27 1.27)) (justify right))
+  )
+  (hierarchical_label "LIN_V" (shape output) (at 81.915 94.615 180) (fields_autoplaced)
+    (effects (font (size 1.27 1.27)) (justify right))
   )
   (hierarchical_label "CURR_U" (shape input) (at 105.41 69.215 180) (fields_autoplaced)
@@
       (effects (font (size 1.27 1.27)))
     )
-    (property "Footprint" "" (at 113.03 92.075 0)
+    (property "Footprint" "Custom:STM32F407G-DISC1-SHIELD" (at 113.03 92.075 0)
       (effects (font (size 1.27 1.27)) hide)
     )
@@
     )
   )
-  (symbol (lib_id "power:+3V0") (at 157.48 66.675 90) (unit 1)
-    (in_bom yes) (on_board yes) (dnp no) (fields_autoplaced)
-    (property "Reference" "#PWR017" (at 161.29 66.675 0)
-      (effects (font (size 1.27 1.27)) hide)
-    )
-    (property "Value" "+3V0" (at 154.305 66.675 90)
-      (effects (font (size 1.27 1.27)) (justify left))
-    )
-    (property "Footprint" "" (at 157.48 66.675 0)
-      (effects (font (size 1.27 1.27)) hide)
-    )
-    (property "Datasheet" "" (at 157.48 66.675 0)
-      (effects (font (size 1.27 1.27)) hide)
-    )
-    (pin "1")
-    (instances
-      (project "Main"
-        (path "/c97a22ab-71f8-4b91-b313-15b8a3e640d7"
-          (reference "#PWR017") (unit 1)
-        )
-        (path "/c97a22ab-71f8-4b91-b313-15b8a3e640d7/9673f451-06b8-4c7c-85a7-44eae9f9c3b1"
-          (reference "#PWR011") (unit 1)
-        )
-      )
-    )
-  )
   (symbol (lib_id "power:GND") (at 106.68 89.535 270) (unit 1)
     (in_bom yes) (on_board yes) (dnp no) (fields_autoplaced)
@@
         )
       )
-    )
-  )
-  (symbol (lib_id "power:+3V0") (at 181.61 66.675 270) (unit 1)
-    (in_bom yes) (on_board yes) (dnp no) (fields_autoplaced)
-    (property "Reference" "#PWR016" (at 177.8 66.675 0)
-      (effects (font (size 1.27 1.27)) hide)
-    )
-    (property "Value" "+3V0" (at 184.785 66.675 90)
-      (effects (font (size 1.27 1.27)) (justify left))
-    )
-    (property "Footprint" "" (at 181.61 66.675 0)
-      (effects (font (size 1.27 1.27)) hide)
-    )
-    (property "Datasheet" "" (at 181.61 66.675 0)
-      (effects (font (size 1.27 1.27)) hide)
-    )
-    (pin "1")
-    (instances
-      (project "Main"
-        (path "/c97a22ab-71f8-4b91-b313-15b8a3e640d7"
-          (reference "#PWR016") (unit 1)
-        )
-        (path "/c97a22ab-71f8-4b91-b313-15b8a3e640d7/9673f451-06b8-4c7c-85a7-44eae9f9c3b1"
-          (reference "#PWR015") (unit 1)
-        )
-      )
