File: MCU.kicad_sch (KiCad schematic)
At the start: 1 part, among them J4 STM32F407G-DISC1-SHIELD

Commit message: update schematics
Connections:
- net +5V: now also J4.53 (5V), J4.54 (5V); no longer J4.2 (VDD), J4.27 (VDD)
- net ADC: now also J4.14 (PA2); no longer J4.32 (PE5)
- net CURR_U: now also J4.7 (PC1); no longer J4.4 (PH0)
- net CURR_V: now also J4.10 (PC2); no longer J4.30 (PC2)
- net CURR_W: now also J4.20 (PC4); no longer J4.35 (PC4)
- net GND: now also J4.100 (GND), J4.2 (GND), J4.23 (GND), J4.49 (GND), J4.5 (GND), J4.51 (GND), J4.52 (GND), J4.99 (GND); no longer J4.12 (PB6), J4.25 (GND), J4.26 (GND), J4.3 (GND)
- net HIN_U: now also J4.27 (PE9); no longer J4.17 (PE15)
- net HIN_V: now also J4.31 (PE13); no longer J4.13 (PE7)
- net HIN_W: now also J4.35 (PB11); no longer J4.18 (PC12)
- net LIN_U: now also J4.25 (PE7); no longer J4.15 (PE11)
- net LIN_V: now also J4.29 (PE11); no longer J4.14 (PE9)
- net LIN_W: now also J4.33 (PE15); no longer J4.16 (PE13)
- net NTC: now also J4.11 (PA1); no longer J4.6 (PE6)
Changed lines of the file:
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@@
   (no_connect (at 129.54 107.315))
   (no_connect (at 158.75 94.615))
-  (no_connect (at 130.81 64.135))
   (no_connect (at 129.54 114.935))
   (no_connect (at 129.54 104.775))
@@
   (no_connect (at 158.75 69.215))
   (no_connect (at 107.95 76.835))
+  (no_connect (at 180.34 86.995))
   (no_connect (at 129.54 69.215))
   (no_connect (at 158.75 79.375))
   (no_connect (at 180.34 81.915))
-  (no_connect (at 106.68 64.135))
   (no_connect (at 129.54 89.535))
   (no_connect (at 158.75 114.935))
@@
   (no_connect (at 180.34 117.475))
   (no_connect (at 158.75 76.835))
+  (no_connect (at 107.95 64.135))
   (no_connect (at 180.34 120.015))
   (no_connect (at 129.54 112.395))
@@
   (no_connect (at 180.34 107.315))
   (no_connect (at 158.75 109.855))
+  (no_connect (at 129.54 64.135))
   (no_connect (at 180.34 99.695))
-  (no_connect (at 181.61 86.995))
   (no_connect (at 158.75 92.075))
   (no_connect (at 158.75 86.995))
-  (wire (pts (xy 129.54 64.135) (xy 130.81 64.135))
-    (stroke (width 0) (type default))
-  )
   (wire (pts (xy 180.34 64.135) (xy 181.61 64.135))
     (stroke (width 0) (type default))
   )
-  (wire (pts (xy 81.915 102.235) (xy 107.95 102.235))
-    (stroke (width 0) (type default))
-  )
   (wire (pts (xy 180.34 122.555) (xy 181.61 122.555))
     (stroke (width 0) (type default))
@@
     (stroke (width 0) (type default))
   )
-  (wire (pts (xy 81.915 97.155) (xy 107.95 97.155))
-    (stroke (width 0) (type default))
-  )
-  (wire (pts (xy 180.34 86.995) (xy 181.61 86.995))
-    (stroke (width 0) (type default))
-  )
   (wire (pts (xy 104.775 74.295) (xy 107.95 74.295))
     (stroke (width 0) (type default))
   )
-  (wire (pts (xy 106.68 64.135) (xy 107.95 64.135))
-    (stroke (width 0) (type default))
-  )
   (wire (pts (xy 129.54 76.835) (xy 132.715 76.835))
     (stroke (width 0) (type default))
   )
+  (wire (pts (xy 93.98 94.615) (xy 107.95 94.615))
+    (stroke (width 0) (type default))
+  )
   (wire (pts (xy 106.68 61.595) (xy 107.95 61.595))
     (stroke (width 0) (type default))
   )
-  (wire (pts (xy 81.915 94.615) (xy 107.95 94.615))
-    (stroke (width 0) (type default))
-  )
   (wire (pts (xy 129.54 71.755) (xy 132.715 71.755))
     (stroke (width 0) (type default))
@@
     (stroke (width 0) (type default))
   )
+  (wire (pts (xy 93.98 92.075) (xy 107.95 92.075))
+    (stroke (width 0) (type default))
+  )
   (wire (pts (xy 157.48 64.135) (xy 158.75 64.135))
     (stroke (width 0) (type default))
@@
     (stroke (width 0) (type default))
   )
+  (wire (pts (xy 93.98 99.695) (xy 107.95 99.695))
+    (stroke (width 0) (type default))
+  )
+  (wire (pts (xy 93.98 97.155) (xy 107.95 97.155))
+    (stroke (width 0) (type default))
+  )
   (wire (pts (xy 106.68 66.675) (xy 107.95 66.675))
     (stroke (width 0) (type default))
   )
-  (wire (pts (xy 81.915 99.695) (xy 107.95 99.695))
-    (stroke (width 0) (type default))
-  )
-  (wire (pts (xy 81.915 92.075) (xy 107.95 92.075))
-    (stroke (width 0) (type default))
-  )
-  (wire (pts (xy 81.915 104.775) (xy 107.95 104.775))
+  (wire (pts (xy 93.98 104.775) (xy 107.95 104.775))
+    (stroke (width 0) (type default))
+  )
+  (wire (pts (xy 93.98 102.235) (xy 107.95 102.235))
     (stroke (width 0) (type default))
   )
@@
     (stroke (width 0) (type default))
   )
-  (hierarchical_label "HIN_W" (shape output) (at 81.915 104.775 180) (fields_autoplaced)
+  (hierarchical_label "HIN_W" (shape output) (at 93.98 104.775 180) (fields_autoplaced)
     (effects (font (size 1.27 1.27)) (justify right))
   )
@@
     (effects (font (size 1.27 1.27)) (justify left))
   )
-  (hierarchical_label "LIN_U" (shape output) (at 81.915 97.155 180) (fields_autoplaced)
-    (effects (font (size 1.27 1.27)) (justify right))
-  )
-  (hierarchical_label "HIN_V" (shape output) (at 81.915 92.075 180) (fields_autoplaced)
+  (hierarchical_label "LIN_U" (shape output) (at 93.98 92.075 180) (fields_autoplaced)
+    (effects (font (size 1.27 1.27)) (justify right))
+  )
+  (hierarchical_label "HIN_V" (shape output) (at 93.98 99.695 180) (fields_autoplaced)
     (effects (font (size 1.27 1.27)) (justify right))
   )
@@
     (effects (font (size 1.27 1.27)) (justify left))
   )
-  (hierarchical_label "LIN_W" (shape output) (at 81.915 99.695 180) (fields_autoplaced)
+  (hierarchical_label "LIN_W" (shape output) (at 93.98 102.235 180) (fields_autoplaced)
     (effects (font (size 1.27 1.27)) (justify right))
   )
@@
     (effects (font (size 1.27 1.27)) (justify left))
   )
-  (hierarchical_label "HIN_U" (shape output) (at 81.915 102.235 180) (fields_autoplaced)
-    (effects (font (size 1.27 1.27)) (justify right))
-  )
-  (hierarchical_label "LIN_V" (shape output) (at 81.915 94.615 180) (fields_autoplaced)
+  (hierarchical_label "HIN_U" (shape output) (at 93.98 94.615 180) (fields_autoplaced)
+    (effects (font (size 1.27 1.27)) (justify right))
+  )
+  (hierarchical_label "LIN_V" (shape output) (at 93.98 97.155 180) (fields_autoplaced)
     (effects (font (size 1.27 1.27)) (justify right))
   )
@@
     (effects (font (size 1.27 1.27)) (justify right))
   )
-  (symbol (lib_name "STM32F407G-DISC1-SHIELD_1") (lib_id "Custom:STM32F407G-DISC1-SHIELD") (at 146.05 92.075 0) (unit 1)
+  (symbol (lib_id "Custom:STM32F407G-DISC1-SHIELD") (at 146.05 92.075 0) (unit 1)
     (in_bom yes) (on_board yes) (dnp no) (fields_autoplaced)
-    (property "Reference" "J4" (at 144.145 53.34 0)
+    (property "Reference" "J4" (at 144.145 53.34 0) (show_name)
       (effects (font (size 1.27 1.27)))
     )
-    (property "Value" "STM32F407G-DISC1-SHIELD" (at 144.145 55.88 0)
+    (property "Value" "STM32F407G-DISC1-SHIELD" (at 144.145 55.88 0) (show_name)
       (effects (font (size 1.27 1.27)))
     )
@@
       (effects (font (size 1.27 1.27)) hide)
     )
-    (pin "1")
+    (pin "55")
     (pin "1")
     (pin "10")
-    (pin "10")
-    (pin "11")
+    (pin "100")
     (pin "11")
     (pin "12")
-    (pin "12")
-    (pin "13")
     (pin "13")
     (pin "14")
-    (pin "14")
-    (pin "15")
     (pin "15")
     (pin "16")
-    (pin "16")
-    (pin "17")
     (pin "17")
     (pin "18")
-    (pin "18")
-    (pin "19")
     (pin "19")
     (pin "2")
-    (pin "2")
-    (pin "20")
     (pin "20")
     (pin "21")
-    (pin "21")
-    (pin "22")
     (pin "22")
     (pin "23")
-    (pin "23")
-    (pin "24")
     (pin "24")
     (pin "25")
-    (pin "25")
-    (pin "26")
     (pin "26")
     (pin "27")
-    (pin "27")
-    (pin "28")
     (pin "28")
     (pin "29")
-    (pin "29")
-    (pin "3")
     (pin "3")
     (pin "30")
-    (pin "30")
-    (pin "31")
     (pin "31")
     (pin "32")
-    (pin "32")
-    (pin "33")
     (pin "33")
     (pin "34")
-    (pin "34")
-    (pin "35")
     (pin "35")
     (pin "36")
-    (pin "36")
-    (pin "37")
     (pin "37")
     (pin "38")
-    (pin "38")
-    (pin "39")
     (pin "39")
     (pin "4")
-    (pin "4")
-    (pin "40")
     (pin "40")
     (pin "41")
-    (pin "41")
-    (pin "42")
     (pin "42")
     (pin "43")
-    (pin "43")
-    (pin "44")
     (pin "44")
     (pin "45")
-    (pin "45")
-    (pin "46")
     (pin "46")
     (pin "47")
-    (pin "47")
-    (pin "48")
     (pin "48")
     (pin "49")
-    (pin "49")
-    (pin "5")
     (pin "5")
     (pin "50")
-    (pin "50")
+    (pin "51")
+    (pin "52")
+    (pin "53")
+    (pin "54")
+    (pin "56")
+    (pin "57")
+    (pin "58")
+    (pin "59")
     (pin "6")
-    (pin "6")
+    (pin "60")
+    (pin "61")
+    (pin "62")
+    (pin "63")
+    (pin "64")
+    (pin "65")
+    (pin "66")
+    (pin "67")
+    (pin "68")
+    (pin "69")
     (pin "7")
-    (pin "7")
+    (pin "70")
+    (pin "71")
+    (pin "72")
+    (pin "73")
+    (pin "74")
+    (pin "75")
+    (pin "76")
+    (pin "77")
+    (pin "78")
+    (pin "79")
     (pin "8")
-    (pin "8")
+    (pin "80")
+    (pin "81")
+    (pin "82")
+    (pin "83")
+    (pin "84")
+    (pin "85")
+    (pin "86")
+    (pin "87")
+    (pin "88")
+    (pin "89")
     (pin "9")
-    (pin "9")
+    (pin "90")
+    (pin "91")
+    (pin "92")
+    (pin "93")
+    (pin "94")
+    (pin "95")
+    (pin "96")
+    (pin "97")
+    (pin "98")
+    (pin "99")
     (instances
       (project "Main"

Commit message: pcb layout design
Connections:
- net HIN_U: now also J4.28 (PE10); no longer J4.27 (PE9)
- net HIN_V: now also J4.32 (PE14); no longer J4.31 (PE13)
- net HIN_W: now also J4.36 (PB12); no longer J4.35 (PB11)
- net LIN_U: now also J4.26 (PE8); no longer J4.25 (PE7)
- net LIN_V: now also J4.30 (PE12); no longer J4.29 (PE11)
- net LIN_W: now also J4.34 (PB10); no longer J4.33 (PE15)
Changed lines of the file:
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@@
   (no_connect (at 158.75 94.615))
   (no_connect (at 129.54 114.935))
-  (no_connect (at 129.54 104.775))
   (no_connect (at 180.34 84.455))
   (no_connect (at 180.34 114.935))
@@
   (no_connect (at 129.54 109.855))
   (no_connect (at 158.75 104.775))
+  (no_connect (at 107.95 97.155))
   (no_connect (at 158.75 117.475))
   (no_connect (at 129.54 81.915))
   (no_connect (at 129.54 120.015))
+  (no_connect (at 107.95 99.695))
   (no_connect (at 158.75 69.215))
   (no_connect (at 107.95 76.835))
@@
   (no_connect (at 158.75 114.935))
   (no_connect (at 158.75 120.015))
+  (no_connect (at 107.95 102.235))
   (no_connect (at 158.75 112.395))
   (no_connect (at 107.95 114.935))
@@
   (no_connect (at 180.34 79.375))
   (no_connect (at 180.34 76.835))
-  (no_connect (at 129.54 97.155))
   (no_connect (at 180.34 109.855))
   (no_connect (at 180.34 94.615))
@@
   (no_connect (at 180.34 92.075))
   (no_connect (at 180.34 112.395))
-  (no_connect (at 129.54 99.695))
   (no_connect (at 107.95 81.915))
   (no_connect (at 129.54 74.295))
@@
   (no_connect (at 158.75 66.675))
   (no_connect (at 107.95 112.395))
-  (no_connect (at 129.54 94.615))
   (no_connect (at 180.34 102.235))
+  (no_connect (at 107.95 92.075))
   (no_connect (at 158.75 84.455))
   (no_connect (at 107.95 109.855))
@@
   (no_connect (at 180.34 71.755))
   (no_connect (at 107.95 86.995))
-  (no_connect (at 129.54 102.235))
   (no_connect (at 180.34 89.535))
   (no_connect (at 158.75 74.295))
   (no_connect (at 129.54 66.675))
   (no_connect (at 129.54 79.375))
+  (no_connect (at 107.95 104.775))
   (no_connect (at 107.95 120.015))
+  (no_connect (at 107.95 94.615))
   (no_connect (at 158.75 71.755))
   (no_connect (at 158.75 99.695))
   (no_connect (at 180.34 97.155))
   (no_connect (at 158.75 97.155))
-  (no_connect (at 129.54 92.075))
   (no_connect (at 180.34 107.315))
   (no_connect (at 158.75 109.855))
@@
   (no_connect (at 158.75 92.075))
   (no_connect (at 158.75 86.995))
+  (wire (pts (xy 130.81 97.155) (xy 129.54 97.155))
+    (stroke (width 0) (type default))
+  )
   (wire (pts (xy 180.34 64.135) (xy 181.61 64.135))
     (stroke (width 0) (type default))
   )
   (wire (pts (xy 180.34 122.555) (xy 181.61 122.555))
+    (stroke (width 0) (type default))
+  )
+  (wire (pts (xy 130.81 94.615) (xy 129.54 94.615))
     (stroke (width 0) (type default))
   )
@@
     (stroke (width 0) (type default))
   )
-  (wire (pts (xy 129.54 76.835) (xy 132.715 76.835))
+  (wire (pts (xy 130.81 104.775) (xy 129.54 104.775))
     (stroke (width 0) (type default))
   )
-  (wire (pts (xy 93.98 94.615) (xy 107.95 94.615))
+  (wire (pts (xy 129.54 76.835) (xy 132.715 76.835))
     (stroke (width 0) (type default))
   )
@@
     (stroke (width 0) (type default))
   )
-  (wire (pts (xy 93.98 92.075) (xy 107.95 92.075))
-    (stroke (width 0) (type default))
-  )
   (wire (pts (xy 157.48 64.135) (xy 158.75 64.135))
     (stroke (width 0) (type default))
@@
     (stroke (width 0) (type default))
   )
-  (wire (pts (xy 93.98 99.695) (xy 107.95 99.695))
+  (wire (pts (xy 130.81 102.235) (xy 129.54 102.235))
     (stroke (width 0) (type default))
   )
-  (wire (pts (xy 93.98 97.155) (xy 107.95 97.155))
+  (wire (pts (xy 130.81 99.695) (xy 129.54 99.695))
     (stroke (width 0) (type default))
   )
@@
     (stroke (width 0) (type default))
   )
-  (wire (pts (xy 93.98 104.775) (xy 107.95 104.775))
-    (stroke (width 0) (type default))
-  )
-  (wire (pts (xy 93.98 102.235) (xy 107.95 102.235))
+  (wire (pts (xy 130.81 92.075) (xy 129.54 92.075))
     (stroke (width 0) (type default))
   )
@@
     (stroke (width 0) (type default))
   )
-  (hierarchical_label "HIN_W" (shape output) (at 93.98 104.775 180) (fields_autoplaced)
-    (effects (font (size 1.27 1.27)) (justify right))
+  (hierarchical_label "HIN_W" (shape output) (at 130.81 104.775 0) (fields_autoplaced)
+    (effects (font (size 1.27 1.27)) (justify left))
   )
   (hierarchical_label "NTC" (shape input) (at 104.775 74.295 180) (fields_autoplaced)
@@
     (effects (font (size 1.27 1.27)) (justify left))
   )
-  (hierarchical_label "LIN_U" (shape output) (at 93.98 92.075 180) (fields_autoplaced)
-    (effects (font (size 1.27 1.27)) (justify right))
+  (hierarchical_label "LIN_U" (shape output) (at 130.81 92.075 0) (fields_autoplaced)
+    (effects (font (size 1.27 1.27)) (justify left))
   )
-  (hierarchical_label "HIN_V" (shape output) (at 93.98 99.695 180) (fields_autoplaced)
-    (effects (font (size 1.27 1.27)) (justify right))
+  (hierarchical_label "HIN_V" (shape output) (at 130.81 99.695 0) (fields_autoplaced)
+    (effects (font (size 1.27 1.27)) (justify left))
   )
   (hierarchical_label "CURR_W" (shape input) (at 132.08 84.455 0) (fields_autoplaced)
     (effects (font (size 1.27 1.27)) (justify left))
   )
-  (hierarchical_label "LIN_W" (shape output) (at 93.98 102.235 180) (fields_autoplaced)
-    (effects (font (size 1.27 1.27)) (justify right))
+  (hierarchical_label "LIN_W" (shape output) (at 130.81 102.235 0) (fields_autoplaced)
+    (effects (font (size 1.27 1.27)) (justify left))
   )
   (hierarchical_label "ADC" (shape input) (at 132.715 76.835 0) (fields_autoplaced)
     (effects (font (size 1.27 1.27)) (justify left))
   )
-  (hierarchical_label "HIN_U" (shape output) (at 93.98 94.615 180) (fields_autoplaced)
-    (effects (font (size 1.27 1.27)) (justify right))
+  (hierarchical_label "HIN_U" (shape output) (at 130.81 94.615 0) (fields_autoplaced)
+    (effects (font (size 1.27 1.27)) (justify left))
   )
-  (hierarchical_label "LIN_V" (shape output) (at 93.98 97.155 180) (fields_autoplaced)
-    (effects (font (size 1.27 1.27)) (justify right))
+  (hierarchical_label "LIN_V" (shape output) (at 130.81 97.155 0) (fields_autoplaced)
+    (effects (font (size 1.27 1.27)) (justify left))
   )
   (hierarchical_label "CURR_U" (shape input) (at 105.41 69.215 180) (fields_autoplaced)
