File: Main.kicad_sch (KiCad schematic)
At the start: 2 parts, among them J5 OUT, J7 AC_IN

Commit message: update schematics
Parts:
- J5: footprint (none) -> Connector_Samtec_HPM_THT:Samtec_HPM-03-01-x-S_Straight_1x03_Pitch5.08mm
- J7: footprint (none) -> Connector_Samtec_HPM_THT:Samtec_HPM-02-01-x-S_Straight_1x02_Pitch5.08mm
Changed lines of the file:
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@@
       (effects (font (size 1.27 1.27)) (justify left))
     )
-    (property "Footprint" "" (at 190.5 78.74 0)
+    (property "Footprint" "Connector_Samtec_HPM_THT:Samtec_HPM-03-01-x-S_Straight_1x03_Pitch5.08mm" (at 190.5 78.74 0)
       (effects (font (size 1.27 1.27)) hide)
     )
@@
       (effects (font (size 1.27 1.27)))
     )
-    (property "Footprint" "" (at 78.105 53.975 0)
+    (property "Footprint" "Connector_Samtec_HPM_THT:Samtec_HPM-02-01-x-S_Straight_1x02_Pitch5.08mm" (at 78.105 53.975 0)
       (effects (font (size 1.27 1.27)) hide)
     )
