File: Rectifier.kicad_sch (KiCad schematic)
At the start: 27 parts, among them J2 Stepdown, J3 Stepdown, J4 Stepdown, J6 Stepdown, SW1 SW_DIP_x01

Commit message: update footprint
Parts:
- removed J2, J3, J4, J6: Stepdown, symbol Connector_Generic:Conn_01x01
- added J8: Conn_01x04, symbol Connector_Generic:Conn_01x04
- D5: footprint (none) -> LED_THT:LED_D5.0mm
- D6: value D_Zener -> DZ24V; footprint (none) -> Diode_THT:D_T-1_P5.08mm_Horizontal
- D7, D8: value D_Zener -> DZ5V; footprint (none) -> Diode_THT:D_T-1_P5.08mm_Horizontal
- R15, R16, R17, R18: footprint (none) -> Resistor_THT:R_Axial_DIN0309_L9.0mm_D3.2mm_P12.70mm_Horizontal
- RV1: footprint (none) -> Varistor:RV_Disc_D7mm_W3.5mm_P5mm
Connections:
- net +15V: now also J8.4 (Pin_4)
- net +24V: now also J8.1 (Pin_1)
- net GND: now also J8.3 (Pin_3)
- net at C33.2, C34.2, D6.2 (A)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: now also J8.2 (Pin_2)

Commit message: update schematics
Parts:
- removed C1: 22uF, symbol Device:C_Polarized_US
- removed C2: 100nF, symbol Device:C
- removed D7: DZ5V, Diode_THT:D_T-1_P5.08mm_Horizontal, symbol Device:D_Zener
- removed F1: Fuse, symbol Device:Fuse
- removed PS1: HLK-10M05, Converter_ACDC:Converter_ACDC_HiLink_HLK-10Mxx, symbol Converter_ACDC:HLK-10M05
- removed SW1: SW_DIP_x01, symbol Switch:SW_DIP_x01
- C31, C34, C36: footprint (none) -> Capacitor_THT:C_Disc_D4.3mm_W1.9mm_P5.00mm
- C32: footprint (none) -> Capacitor_THT:CP_Radial_D30.0mm_P10.00mm_SnapIn
- C33, C35: footprint (none) -> Capacitor_THT:CP_Radial_D5.0mm_P2.50mm
- J8: footprint (none) -> Connector_Samtec_HPM_THT:Samtec_HPM-04-01-x-S_Straight_1x04_Pitch5.08mm
Connections:
- net N is gone; now on net L: BR1.3 (~_2), PS2.2 (AC/N), PS3.2 (AC/N), RV1.2
- net L: now also PS2.1 (AC/L), RV1.1
- net at BR1.2 (~_1), PS3.1 (AC/L): no longer PS2.1 (AC/L), RV1.1
Other:
- moved on the sheet: C33, C34, D6, J8, PS2, RV1

Commit message: pcb layout design
Connections:
- net L: now also BR1.2 (~_1), PS3.1 (AC/L); no longer BR1.3 (~_2), PS2.2 (AC/N), PS3.2 (AC/N), RV1.2
- new net N: BR1.3 (~_2), PS2.2 (AC/N), PS3.2 (AC/N), RV1.2
Other:
- moved on the sheet: RV1
Changed lines of the file:
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@@
   (junction (at 74.93 85.09) (diameter 0) (color 0 0 0 0)
   )
+  (junction (at 80.645 41.91) (diameter 0) (color 0 0 0 0)
+  )
   (junction (at 121.92 70.485) (diameter 0) (color 0 0 0 0)
   )
   (junction (at 134.62 41.91) (diameter 0) (color 0 0 0 0)
   )
-  (junction (at 79.375 75.565) (diameter 0) (color 0 0 0 0)
-  )
   (junction (at 146.685 49.53) (diameter 0) (color 0 0 0 0)
   )
@@
   (junction (at 121.92 49.53) (diameter 0) (color 0 0 0 0)
   )
-  (junction (at 79.375 41.91) (diameter 0) (color 0 0 0 0)
-  )
   (junction (at 63.5 50.8) (diameter 0) (color 0 0 0 0)
   )
@@
   (junction (at 134.62 78.105) (diameter 0) (color 0 0 0 0)
   )
+  (junction (at 80.645 70.485) (diameter 0) (color 0 0 0 0)
+  )
   (junction (at 134.62 49.53) (diameter 0) (color 0 0 0 0)
   )
@@
     (stroke (width 0) (type default))
   )
+  (wire (pts (xy 80.645 41.91) (xy 89.535 41.91))
+    (stroke (width 0) (type default))
+  )
   (wire (pts (xy 74.93 130.175) (xy 74.93 133.985))
     (stroke (width 0) (type default))
   )
-  (wire (pts (xy 31.115 70.485) (xy 89.535 70.485))
+  (wire (pts (xy 31.115 70.485) (xy 80.645 70.485))
     (stroke (width 0) (type default))
   )
@@
     (stroke (width 0) (type default))
   )
-  (wire (pts (xy 79.375 75.565) (xy 85.09 75.565))
-    (stroke (width 0) (type default))
-  )
   (wire (pts (xy 121.92 78.105) (xy 134.62 78.105))
     (stroke (width 0) (type default))
@@
     (stroke (width 0) (type default))
   )
-  (wire (pts (xy 63.5 41.91) (xy 63.5 42.545))
+  (wire (pts (xy 80.645 70.485) (xy 89.535 70.485))
+    (stroke (width 0) (type default))
+  )
+  (wire (pts (xy 63.5 41.91) (xy 63.5 43.18))
     (stroke (width 0) (type default))
   )
@@
     (stroke (width 0) (type default))
   )
-  (wire (pts (xy 63.5 41.91) (xy 79.375 41.91))
-    (stroke (width 0) (type default))
-  )
   (wire (pts (xy 109.855 41.91) (xy 121.92 41.91))
     (stroke (width 0) (type default))
@@
     (stroke (width 0) (type default))
   )
-  (wire (pts (xy 79.375 41.91) (xy 89.535 41.91))
+  (wire (pts (xy 63.5 41.91) (xy 80.645 41.91))
     (stroke (width 0) (type default))
   )
@@
     (stroke (width 0) (type default))
   )
-  (wire (pts (xy 63.5 50.8) (xy 63.5 50.165))
-    (stroke (width 0) (type default))
-  )
-  (wire (pts (xy 79.375 41.91) (xy 79.375 75.565))
-    (stroke (width 0) (type default))
-  )
   (wire (pts (xy 146.685 49.53) (xy 169.545 49.53))
     (stroke (width 0) (type default))
@@
     (stroke (width 0) (type default))
   )
+  (wire (pts (xy 80.645 41.91) (xy 80.645 70.485))
+    (stroke (width 0) (type default))
+  )
   (wire (pts (xy 134.62 49.53) (xy 146.685 49.53))
     (stroke (width 0) (type default))
   )
-  (wire (pts (xy 27.94 75.565) (xy 79.375 75.565))
+  (wire (pts (xy 27.94 75.565) (xy 85.09 75.565))
     (stroke (width 0) (type default))
   )
@@
     )
   )
-  (symbol (lib_id "Device:Varistor") (at 63.5 46.355 0) (unit 1)
-    (in_bom yes) (on_board yes) (dnp no) (fields_autoplaced)
-    (property "Reference" "RV1" (at 66.675 45.2783 0)
-      (effects (font (size 1.27 1.27)) (justify left))
-    )
-    (property "Value" "Varistor" (at 66.675 47.8183 0)
-      (effects (font (size 1.27 1.27)) (justify left))
-    )
-    (property "Footprint" "Varistor:RV_Disc_D7mm_W3.5mm_P5mm" (at 61.722 46.355 90)
-      (effects (font (size 1.27 1.27)) hide)
-    )
-    (property "Datasheet" "~" (at 63.5 46.355 0)
-      (effects (font (size 1.27 1.27)) hide)
-    )
-    (property "Sim.Name" "kicad_builtin_varistor" (at 63.5 46.355 0)
-      (effects (font (size 1.27 1.27)) hide)
-    )
-    (property "Sim.Device" "SUBCKT" (at 63.5 46.355 0)
-      (effects (font (size 1.27 1.27)) hide)
-    )
-    (property "Sim.Pins" "1=A 2=B" (at 63.5 46.355 0)
-      (effects (font (size 1.27 1.27)) hide)
-    )
-    (property "Sim.Params" "threshold=1k" (at 63.5 46.355 0)
-      (effects (font (size 1.27 1.27)) hide)
-    )
-    (property "Sim.Library" "${KICAD7_SYMBOL_DIR}/Simulation_SPICE.sp" (at 63.5 46.355 0)
-      (effects (font (size 1.27 1.27)) hide)
-    )
+  (symbol (lib_id "Device:Varistor") (at 63.5 46.99 0) (unit 1)
+    (in_bom yes) (on_board yes) (dnp no) (fields_autoplaced)
+    (property "Reference" "RV1" (at 66.675 45.9133 0)
+      (effects (font (size 1.27 1.27)) (justify left))
+    )
+    (property "Value" "Varistor" (at 66.675 48.4533 0)
+      (effects (font (size 1.27 1.27)) (justify left))
+    )
+    (property "Footprint" "Varistor:RV_Disc_D7mm_W3.5mm_P5mm" (at 61.722 46.99 90)
+      (effects (font (size 1.27 1.27)) hide)
+    )
+    (property "Datasheet" "~" (at 63.5 46.99 0)
+      (effects (font (size 1.27 1.27)) hide)
+    )
+    (property "Sim.Name" "kicad_builtin_varistor" (at 63.5 46.99 0)
+      (effects (font (size 1.27 1.27)) hide)
+    )
+    (property "Sim.Device" "SUBCKT" (at 63.5 46.99 0)
+      (effects (font (size 1.27 1.27)) hide)
+    )
+    (property "Sim.Pins" "1=A 2=B" (at 63.5 46.99 0)
+      (effects (font (size 1.27 1.27)) hide)
+    )
+    (property "Sim.Params" "threshold=1k" (at 63.5 46.99 0)
+      (effects (font (size 1.27 1.27)) hide)
+    )
+    (property "Sim.Library" "${KICAD7_SYMBOL_DIR}/Simulation_SPICE.sp" (at 63.5 46.99 0)
+      (effects (font (size 1.27 1.27)) hide)
+    )
