File: Main.kicad_pcb (KiCad board)
At the start: 2 copper layers, 65 parts, among them IC1 STGIPQ3H60T-HL, IC2 ACS724LLCTR-05AU-T, IC3 ACS724LLCTR-05AU-T, IC4 ACS724LLCTR-05AU-T, J1 STM32F407G-DISC1-SHIELD, J5 OUT, J7 AC_IN, J8 Conn_01x04

Commit message: pcb layout design
Parts:
- C10, C11, C12, C13, C14, C15, C9: footprint Capacitor_THT:C_Disc_D4.3mm_W1.9mm_P5.00mm -> Capacitor_SMD:C_0805_2012Metric; moved to B.Cu
- IC1: moved to F.Cu
- IC2, IC3, IC4: moved to B.Cu
- PS 24VDC: renamed from PS2
- PS 5VDC: renamed from PS3
- moved C32 180.5 mm to (77.4, 130.8), turned to 90 degrees
- moved J7 168.1 mm to (51.9, 69.2), turned to 180 degrees
- moved RV1 156.0 mm to (50.9, 78.1), turned to -90 degrees
- moved BR1 148.1 mm to (50.9, 107.5), turned to -90 degrees
- moved D5 147.0 mm to (100.8, 114.1)
- moved C31 145.7 mm to (96.9, 124.8), turned to 90 degrees
- moved R15 143.5 mm to (106.9, 128.6)
- moved C35 139.9 mm to (114.6, 84.2), turned to 90 degrees
- moved C33 139.7 mm to (114.7, 75.6), turned to 90 degrees
- moved R17 136.5 mm to (106.9, 117.5)
- moved R16 127.8 mm to (119.6, 123.0), turned to 180 degrees
- moved IC1 126.5 mm to (158.3, 97.6), turned to 180 degrees
- moved D6 125.9 mm to (120.9, 77.2), turned to 90 degrees
- moved D8 125.6 mm to (120.9, 85.9), turned to 90 degrees
- moved R18 121.6 mm to (119.6, 112.1), turned to 180 degrees
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Connections:
- BR1 pad 2: Net-(BR1-~_1) -> /Rectifier & Power supply/L
- BR1 pad 3: /Rectifier & Power supply/L -> /Rectifier & Power supply/N
- J1 pad 25: /Inverter/LIN_U -> unconnected-(J1-PE7-Pad25)
- J1 pad 26: unconnected-(J1-PE8-Pad26) -> /Inverter/LIN_U
- J1 pad 27: /Inverter/HIN_U -> unconnected-(J1-PE9-Pad27)
- J1 pad 28: unconnected-(J1-PE10-Pad28) -> /Inverter/HIN_U
- J1 pad 29: /Inverter/LIN_V -> unconnected-(J1-PE11-Pad29)
- J1 pad 30: unconnected-(J1-PE12-Pad30) -> /Inverter/LIN_V
- J1 pad 31: /Inverter/HIN_V -> unconnected-(J1-PE13-Pad31)
- J1 pad 32: unconnected-(J1-PE14-Pad32) -> /Inverter/HIN_V
- J1 pad 33: /Inverter/LIN_W -> unconnected-(J1-PE15-Pad33)
- J1 pad 34: unconnected-(J1-PB10-Pad34) -> /Inverter/LIN_W
- J1 pad 35: /Inverter/HIN_W -> unconnected-(J1-PB11-Pad35)
- J1 pad 36: unconnected-(J1-PB12-Pad36) -> /Inverter/HIN_W
- J7 pad 1: /Rectifier & Power supply/L -> /Rectifier & Power supply/N
- PS 24VDC pad 2: /Rectifier & Power supply/L -> /Rectifier & Power supply/N
- PS 5VDC pad 1: Net-(BR1-~_1) -> /Rectifier & Power supply/L
- PS 5VDC pad 2: /Rectifier & Power supply/L -> /Rectifier & Power supply/N
- RV1 pad 2: /Rectifier & Power supply/L -> /Rectifier & Power supply/N
Routing:
- net GND: track 100.6 -> 802.4 mm, vias 0 -> 8
- net +5V: track 0.00 -> 224.2 mm, vias 0 -> 10
- net /Inverter/CURR_U: track 0.00 -> 193.9 mm, vias 0 -> 2
- net /Inverter/CURR_V: track 0.00 -> 162.4 mm, vias 0 -> 2
- net /Inverter/CURR_W: track 0.00 -> 145.6 mm, vias 0 -> 2
- net /Inverter/HV: track 0.00 -> 114.6 mm
- net Net-(IC1-NU): track 0.00 -> 105.7 mm
- net RS: track 0.00 -> 103.3 mm, vias 0 -> 2
- net /Rectifier & Power supply/L: track 0.00 -> 96.2 mm
- net +15V: track 0.00 -> 95.2 mm, vias 0 -> 2
- net /Rectifier & Power supply/N: track 0.00 -> 92.0 mm
- net Net-(IC1-OP+): track 0.00 -> 72.6 mm, vias 0 -> 2
- net Net-(D6-A): track 0.00 -> 65.6 mm
- net +24V: track 0.00 -> 55.7 mm, vias 0 -> 2
- net /Inverter/LIN_U: track 16.4 -> 64.7 mm
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- added copper zone on B.Cu, net GND
- added copper zone on F.Cu, net GND
Other:
- board outline added: 229.1 x 127.9 mm
- board text added: "AC Induction Motor Control Board Muhammad Lukmanul Hakim 5022201237 Control & Automation Laboratory Electrical Engineering ITS Supported by PT Infoglobal Teknologi Semesta"
- board text added: "WARNING! HIGH VOLTAGE ON BOARD"

Commit message: add copper zone, drill mounting, text to the pcb
Parts:
- moved R1 2.01 mm to (185.8, 113.5)
Routing:
- net /Inverter/NTC: track 120.0 -> 121.7 mm
- net +5V: track 224.2 -> 225.5 mm
- added copper zone on B.Cu, net (none)
- added copper zone on F.Cu, net (none)
- removed copper zone on B.Cu, net GND
- removed copper zone on F.Cu, net GND
